Commit message: Feat 完善实现基本gazebo中导航功能

File: fn_sim/Fines_Gazebo_Simulator/urdf/robot.urdf (robot description, URDF)
Before this commit: robot FINES, 2 links, 1 joints
Links:
- link base_link: geometry collision box size=0.25 0.125 0.0625; visual box size=0.25 0.125 0.0625
Joints:
- joint lidar_joint: origin xyz=0.8 0 0.5 rpy=0 0 0 -> xyz=0.1 0 0.1 rpy=0 0 0

Commit message: feat: 更换了场景以及机器人模型
存在问题1: 四轮机器人动力模型缺陷，计划改用三轮机器人
2： 雷达安装位置并不合适

File: fn_sim/Fines_Gazebo_Simulator/urdf/robot.urdf (robot description, URDF)
Before this commit: robot FINES, 2 links, 1 joints
Links:
- added link base_origin
- added link left_front_wheel, mass 1e-5; visual cylinder length=0.1 radius=0.15
- added link left_rear_wheel, mass 1e-5; visual cylinder length=0.1 radius=0.15
- added link right_front_wheel, mass 1e-5; visual cylinder length=0.1 radius=0.15
- added link right_rear_wheel, mass 1e-5; visual cylinder length=0.1 radius=0.15
- link base_lidar: mass 0.1 -> 1e-5; geometry visual cylinder length=0.35 radius=0.03
- link base_link: mass 1.0 -> 1e-5; geometry visual box size=0.6 0.4 0.3
Joints:
- removed joint lidar_joint
- added joint base_lidar_joint: type fixed, parent base_link, child base_lidar, origin xyz=0.0 0 0.6 rpy=0 0 0
- added joint base_link_joint: type fixed, parent base_origin, child base_link, origin xyz=0.0 0 -0.5 rpy=0 0 0
- added joint left_front_joint: type fixed, parent base_link, child left_front_wheel, origin xyz=0.2 -0.25 -0.1 rpy=1.57 0 0
- added joint left_rear_joint: type fixed, parent base_link, child left_rear_wheel, origin xyz=-0.2 -0.25 -0.1 rpy=1.57 0 0
- added joint right_rear_joint: type fixed, parent base_link, child right_rear_wheel, origin xyz=-0.2 0.25 -0.1 rpy=-1.57 0 0
- added joint rigth_front_joint: type fixed, parent base_link, child right_front_wheel, origin xyz=0.2 0.25 -0.1 rpy=-1.57 0 0

Commit message: feat: 解为万向轮决了四轮驱动的问题，修改

File: fn_sim/Fines_Gazebo_Simulator/urdf/robot.urdf (robot description, URDF)
Before this commit: robot example, 7 links, 6 joints
Links:
- link base_lidar: geometry visual cylinder length=0.6 radius=0.03
Joints:
- removed joint rigth_front_joint
- added joint right_front_joint: type fixed, parent base_link, child right_front_wheel, origin xyz=0.2 0.25 -0.1 rpy=-1.57 0 0
- joint base_lidar_joint: origin xyz=0.0 0 0.6 rpy=0 0 0 -> xyz=0.0 0 0.6 rpy=3.14159 0 0

Commit message: feat: 初步完成了Mapmanager对Localmap的可视化功能，TODO：测试Localmap的各功能

File: fn_sim/Fines_Gazebo_Simulator/urdf/robot.urdf (robot description, URDF)
Before this commit: robot example, 7 links, 6 joints
Joints:
- joint base_lidar_joint: origin xyz=0.0 0 0.6 rpy=3.14159 0 0 -> xyz=0.0 0 0.85 rpy=0 0 0
- joint base_link_joint: origin xyz=0.0 0 -0.5 rpy=0 0 0 -> xyz=0.0 0 -0.75 rpy=0 0 0
- joint left_front_joint: origin xyz=0.2 -0.25 -0.1 rpy=1.57 0 0 -> xyz=0.2 -0.25 0.15 rpy=1.57 0 0
- joint left_rear_joint: origin xyz=-0.2 -0.25 -0.1 rpy=1.57 0 0 -> xyz=-0.2 -0.25 0.15 rpy=1.57 0 0
- joint right_front_joint: origin xyz=0.2 0.25 -0.1 rpy=-1.57 0 0 -> xyz=0.2 0.25 0.15 rpy=-1.57 0 0
- joint right_rear_joint: origin xyz=-0.2 0.25 -0.1 rpy=-1.57 0 0 -> xyz=-0.2 0.25 0.15 rpy=-1.57 0 0

Commit message: feat: 完善配置

File: fn_sim/Fines_Gazebo_Simulator/urdf/robot.urdf (robot description, URDF)
Before this commit: robot example, 7 links, 6 joints
Links:
- link base_lidar: geometry visual cylinder length=0.25 radius=0.03
Joints:
- joint base_lidar_joint: origin xyz=0.0 0 0.85 rpy=0 0 0 -> xyz=0.0 0 0.40 rpy=0 0 0
